Commit message: Modified urdf to replace kinova gripper with robotiq 85 gripper; MoveIt! configuration not yet updated...

File: kinova_description/urdf/j2s7s300.xacro (robot description, xacro)
@@ -16,4 +16,5 @@
     <xacro:include filename="$(find kinova_description)/urdf/kinova_common.xacro" />
     <xacro:include filename="$(find kinova_description)/urdf/kinova_finger_set.xacro" />
+    <xacro:include filename="$(find robotiq_85_description)/urdf/robotiq_85_gripper.urdf.xacro" />
     <!-- Import all Gazebo-customization elements -->
     <xacro:include filename="$(find kinova_description)/urdf/kinova.gazebo" />
@@ -115,4 +116,5 @@
         <xacro:kinova_armlink link_name="${prefix}_link_6" link_mesh="${link_6_mesh}" use_ring_mesh="true" ring_mesh="ring_small" mesh_no="${link_6_mesh_no}"/>
         <xacro:kinova_armjoint joint_name="${prefix}_joint_6" type="${joint_6_type}" parent="${prefix}_link_5" child="${prefix}_link_6" joint_axis_xyz="${joint_6_axis_xyz}" joint_origin_xyz="${joint_6_origin_xyz}" joint_origin_rpy="${joint_6_origin_rpy}" joint_lower_limit="${joint_6_lower_limit}" joint_upper_limit="${joint_6_upper_limit}"/>
+        <!--
         <xacro:kinova_armlink link_name="${prefix}_link_7" link_mesh="${link_7_mesh}" use_ring_mesh="true" ring_mesh="ring_small" mesh_no="${link_7_mesh_no}"/>
         <xacro:kinova_armjoint joint_name="${prefix}_joint_7" type="${joint_7_type}" parent="${prefix}_link_6" child="${prefix}_link_7" joint_axis_xyz="${joint_7_axis_xyz}" joint_origin_xyz="${joint_7_origin_xyz}" joint_origin_rpy="${joint_7_origin_rpy}" joint_lower_limit="${joint_7_lower_limit}" joint_upper_limit="${joint_7_upper_limit}"/>
@@ -120,4 +122,50 @@
         <xacro:kinova_virtual_joint joint_name="${prefix}_joint_end_effector" type="${joint_end_effector_type}" parent="${prefix}_link_7" child="${prefix}_end_effector" joint_axis_xyz="${joint_end_effector_axis_xyz}" joint_origin_xyz="${joint_end_effector_origin_xyz}" joint_origin_rpy="${joint_end_effector_origin_rpy}" joint_lower_limit="0" joint_upper_limit="0"/>
         <xacro:kinova_3fingers link_hand="${prefix}_link_7" prefix="${prefix}_"/>
+        -->
+        <!-- RAIL end-effector additions/modifications -->
+        <joint name="${prefix}_joint_7" type="continuous">
+          <parent link="${prefix}_link_6" />
+          <child link = "${prefix}_link_7" />
+          <origin xyz="0 0.06075 0" rpy="${J_PI/2} 0 0" />
+          <axis xyz="0 0 1" />
+          <limit effort="600.8" velocity="0.785"/>
+          <dynamics damping="0.0" friction="0.0"/>
+        </joint>
+        <link name="${prefix}_link_7">
+          <visual>
+            <geometry>
+              <mesh filename="package://kinova_description/meshes/wrist_3.dae"/>
+            </geometry>
+          </visual>
+          <collision>
+            <geometry>
+              <mesh filename="package://kinova_description/meshes/wrist_3.stl"/>
+            </geometry>
+          </collision>
+        </link>
+        <joint name="${prefix}_ee_fixed_joint" type="fixed">
+          <parent link="${prefix}_link_7" />
+          <child link = "${prefix}_ee_base" />
+          <origin xyz="0 0 -0.09380704" rpy="0 ${J_PI/2} 0" />
+        </joint>
+        <link name="${prefix}_ee_base"/>
+        <joint name="${prefix}_ee_gripper" type="fixed">
+          <parent link="${prefix}_ee_base" />
+          <child link ="${prefix}_ee_link" />
+          <origin xyz="0.13 0 0" />
+        </joint>
+        <link name="${prefix}_ee_link"/>
+        <transmission name="${prefix}_joint_7_trans">
+          <type>transmission_interface/SimpleTransmission</type>
+          <joint name="${prefix}_joint_7">
+            <hardwareInterface>PositionJointInterface</hardwareInterface>
+          </joint>
+          <actuator name="${prefix}_joint_7_motor">
+            <mechanicalReduction>1</mechanicalReduction>
+          </actuator>
+        </transmission>
+        <xacro:robotiq_85_gripper prefix="${prefix}_" parent="${prefix}_ee_base">
+          <origin xyz="0 0 0" rpy="0 0 0" />
+        </xacro:robotiq_85_gripper>
     </xacro:macro>
 </root>

Commit message: moved arm origin

File: kinova_description/urdf/j2s7s300.xacro (robot description, xacro)
@@ -41,6 +41,6 @@
     <property name="joint_base_type" value="fixed" />
     <property name="joint_base_axis_xyz" value="0 0 0" />
-    <property name="joint_base_origin_xyz" value="0 0 0" />
-    <property name="joint_base_origin_rpy" value="0 ${J_PI/2} 0" />
+    <property name="joint_base_origin_xyz" value="0.06079866 0 0" />
+    <property name="joint_base_origin_rpy" value="${J_PI/2} 0 ${J_PI/2}" />
     <property name="joint_1" value="joint_1" />
     <property name="joint_1_type" value="continuous" />
@@ -98,5 +98,5 @@
     <property name="joint_end_effector_origin_rpy" value="${J_PI} 0 0" />
     <!--xacro:macro name="jaco_robot" params="parent prefix"-->
-    <xacro:macro name="j2s7s300" params="base_parent prefix:=j2s7s300">
+    <xacro:macro name="j2s7s300" params="base_parent prefix:=j2s7s300 *origin">
         <xacro:gazebo_config robot_namespace="${prefix}"/>
         <xacro:kinova_armlink link_name="${prefix}_link_base" link_mesh="${link_base_mesh}" mesh_no="${link_base_mesh_no}"/>

Commit message: make the kinova robot urdf more general

File: kinova_description/urdf/j2s7s300.xacro (robot description, xacro)
@@ -41,6 +41,4 @@
     <property name="joint_base_type" value="fixed" />
     <property name="joint_base_axis_xyz" value="0 0 0" />
-    <property name="joint_base_origin_xyz" value="0.06079866 0 0" />
-    <property name="joint_base_origin_rpy" value="${J_PI/2} 0 ${J_PI/2}" />
     <property name="joint_1" value="joint_1" />
     <property name="joint_1_type" value="continuous" />
@@ -98,8 +96,8 @@
     <property name="joint_end_effector_origin_rpy" value="${J_PI} 0 0" />
     <!--xacro:macro name="jaco_robot" params="parent prefix"-->
-    <xacro:macro name="j2s7s300" params="base_parent prefix:=j2s7s300 *origin">
+    <xacro:macro name="j2s7s300" params="base_parent prefix:=j2s7s300 trans rot">
         <xacro:gazebo_config robot_namespace="${prefix}"/>
         <xacro:kinova_armlink link_name="${prefix}_link_base" link_mesh="${link_base_mesh}" mesh_no="${link_base_mesh_no}"/>
-        <xacro:kinova_armjoint joint_name="${prefix}_joint_base" type="${joint_base_type}" parent="${base_parent}" child="${prefix}_link_base" joint_axis_xyz="${joint_base_axis_xyz}" joint_origin_xyz="${joint_base_origin_xyz}" joint_origin_rpy="${joint_base_origin_rpy}" joint_lower_limit="0" joint_upper_limit="0" fixed="true"/>
+        <xacro:kinova_armjoint joint_name="${prefix}_joint_base" type="${joint_base_type}" parent="${base_parent}" child="${prefix}_link_base" joint_axis_xyz="${joint_base_axis_xyz}" joint_origin_xyz="${trans}" joint_origin_rpy="${rot}" joint_lower_limit="0" joint_upper_limit="0" fixed="true"/>
         <xacro:kinova_armlink link_name="${prefix}_link_1" link_mesh="${link_1_mesh}" use_ring_mesh="true" mesh_no="${link_1_mesh_no}"/>
         <xacro:kinova_armjoint joint_name="${prefix}_joint_1" type="${joint_1_type}" parent="${prefix}_link_base" child="${prefix}_link_1" joint_axis_xyz="${joint_1_axis_xyz}" joint_origin_xyz="${joint_1_origin_xyz}" joint_origin_rpy="${joint_1_origin_rpy}" joint_lower_limit="${joint_1_lower_limit}" joint_upper_limit="${joint_1_upper_limit}"/>

Commit message: switched to using robotiq_85_description package for gripper; added default values to j2s7s300 base rotation and translation; removed j2s7s300 prefix from gripper links (as they're already adequately prefixed with robotiq85_gripper)

File: kinova_description/urdf/j2s7s300.xacro (robot description, xacro)
@@ -15,5 +15,5 @@
     xmlns:xacro="http://ros.org/wiki/xacro">
     <xacro:include filename="$(find kinova_description)/urdf/kinova_common.xacro" />
-    <xacro:include filename="$(find vector_description)/urdf/manipulation/robotiq/robotiq_85_gripper.urdf.xacro" />
+    <xacro:include filename="$(find robotiq_85_description)/urdf/robotiq_85_gripper.urdf.xacro" />
     <property name="link_base_mesh" value="base" />
     <property name="link_1_mesh" value="shoulder" />
@@ -96,5 +96,7 @@
     <property name="joint_end_effector_origin_rpy" value="${J_PI} 0 0" />
     <!--xacro:macro name="jaco_robot" params="parent prefix"-->
-    <xacro:macro name="j2s7s300" params="base_parent prefix:=j2s7s300 trans rot">
+    <property name="default_base_trans" value="0 0 0" />
+    <property name="default_base_rot" value="0 0 0" />
+    <xacro:macro name="j2s7s300" params="base_parent prefix:=j2s7s300 trans:=${default_base_trans} rot:=${default_base_rot}">
         <xacro:gazebo_config robot_namespace="${prefix}"/>
         <xacro:kinova_armlink link_name="${prefix}_link_base" link_mesh="${link_base_mesh}" mesh_no="${link_base_mesh_no}"/>
@@ -161,5 +163,5 @@
           </actuator>
         </transmission>
-        <xacro:robotiq_85_gripper prefix="${prefix}_" parent="${prefix}_ee_base">
+        <xacro:robotiq_85_gripper prefix="" parent="${prefix}_ee_base">
           <origin xyz="0 0 0" rpy="0 0 0" />
         </xacro:robotiq_85_gripper>

Commit message: Parameter changes for poli

File: kinova_description/urdf/j2s7s300.xacro (robot description, xacro)
@@ -16,4 +16,6 @@
     <xacro:include filename="$(find kinova_description)/urdf/kinova_common.xacro" />
     <xacro:include filename="$(find robotiq_85_description)/urdf/robotiq_85_gripper.urdf.xacro" />
+    <!-- Import all Gazebo-customization elements -->
+    <xacro:include filename="$(find kinova_description)/urdf/kinova.gazebo" />
     <property name="link_base_mesh" value="base" />
     <property name="link_1_mesh" value="shoulder" />

File: kinova_description/urdf/kinova_common.xacro (robot description, xacro)
@@ -14,5 +14,5 @@
 	xmlns:xacro="http://ros.org/wiki/xacro">
 <xacro:include filename="$(find kinova_description)/urdf/kinova_inertial.xacro" />
-    <property name="J_PI" value="3.1415926535897931" />
+    <xacro:property name="J_PI" value="3.1415926535897931" />
     <xacro:macro name="kinova_armlink" params="link_name link_mesh ring_mesh:=ring_big use_ring_mesh:=false mesh_no">
         <link name="${link_name}">

Commit message: updated urdf to use jaco gripper

File: kinova_description/urdf/j2s7s300.xacro (robot description, xacro)
@@ -15,5 +15,7 @@
     xmlns:xacro="http://ros.org/wiki/xacro">
     <xacro:include filename="$(find kinova_description)/urdf/kinova_common.xacro" />
-    <xacro:include filename="$(find vector_description)/urdf/manipulation/robotiq/robotiq_85_gripper.urdf.xacro" />
+    <xacro:include filename="$(find robotiq_85_description)/urdf/robotiq_85_gripper.urdf.xacro" />
+    <!-- Import all Gazebo-customization elements -->
+    <xacro:include filename="$(find kinova_description)/urdf/kinova.gazebo" />
     <property name="link_base_mesh" value="base" />
     <property name="link_1_mesh" value="shoulder" />
@@ -41,6 +43,4 @@
     <property name="joint_base_type" value="fixed" />
     <property name="joint_base_axis_xyz" value="0 0 0" />
-    <property name="joint_base_origin_xyz" value="0.06079866 0 0" />
-    <property name="joint_base_origin_rpy" value="${J_PI/2} 0 ${J_PI/2}" />
     <property name="joint_1" value="joint_1" />
     <property name="joint_1_type" value="continuous" />
@@ -98,8 +98,10 @@
     <property name="joint_end_effector_origin_rpy" value="${J_PI} 0 0" />
     <!--xacro:macro name="jaco_robot" params="parent prefix"-->
-    <xacro:macro name="j2s7s300" params="base_parent prefix:=j2s7s300 *origin">
+    <property name="default_base_trans" value="0 0 0" />
+    <property name="default_base_rot" value="0 0 0" />
+    <xacro:macro name="j2s7s300" params="base_parent prefix:=j2s7s300 trans:=${default_base_trans} rot:=${default_base_rot}">
         <xacro:gazebo_config robot_namespace="${prefix}"/>
         <xacro:kinova_armlink link_name="${prefix}_link_base" link_mesh="${link_base_mesh}" mesh_no="${link_base_mesh_no}"/>
-        <xacro:kinova_armjoint joint_name="${prefix}_joint_base" type="${joint_base_type}" parent="${base_parent}" child="${prefix}_link_base" joint_axis_xyz="${joint_base_axis_xyz}" joint_origin_xyz="${joint_base_origin_xyz}" joint_origin_rpy="${joint_base_origin_rpy}" joint_lower_limit="0" joint_upper_limit="0" fixed="true"/>
+        <xacro:kinova_armjoint joint_name="${prefix}_joint_base" type="${joint_base_type}" parent="${base_parent}" child="${prefix}_link_base" joint_axis_xyz="${joint_base_axis_xyz}" joint_origin_xyz="${trans}" joint_origin_rpy="${rot}" joint_lower_limit="0" joint_upper_limit="0" fixed="true"/>
         <xacro:kinova_armlink link_name="${prefix}_link_1" link_mesh="${link_1_mesh}" use_ring_mesh="true" mesh_no="${link_1_mesh_no}"/>
         <xacro:kinova_armjoint joint_name="${prefix}_joint_1" type="${joint_1_type}" parent="${prefix}_link_base" child="${prefix}_link_1" joint_axis_xyz="${joint_1_axis_xyz}" joint_origin_xyz="${joint_1_origin_xyz}" joint_origin_rpy="${joint_1_origin_rpy}" joint_lower_limit="${joint_1_lower_limit}" joint_upper_limit="${joint_1_upper_limit}"/>
@@ -163,5 +165,5 @@
           </actuator>
         </transmission>
-        <xacro:robotiq_85_gripper prefix="${prefix}_" parent="${prefix}_ee_base">
+        <xacro:robotiq_85_gripper prefix="" parent="${prefix}_ee_base">
           <origin xyz="0 0 0" rpy="0 0 0" />
         </xacro:robotiq_85_gripper>

Commit message: Rotate robotiq gripper to match physical hardware

File: kinova_description/urdf/j2s7s300.xacro (robot description, xacro)
@@ -166,5 +166,5 @@
         </transmission>
         <xacro:robotiq_85_gripper prefix="" parent="${prefix}_ee_base">
-          <origin xyz="0 0 0" rpy="0 0 0" />
+          <origin xyz="0 0 0" rpy="${J_PI/2} 0 0"/>
         </xacro:robotiq_85_gripper>
     </xacro:macro>

Commit message: Fixing arm driver boot issues

File: kinova_description/urdf/j2s7s300.xacro (robot description, xacro)
@@ -99,4 +99,6 @@
     <xacro:property name="joint_end_effector_origin_xyz" value="0 0 -0.1600" />
     <xacro:property name="joint_end_effector_origin_rpy" value="${J_PI} 0 0" />
+    <xacro:property name="default_base_trans" value="0 0 0"/>
+    <xacro:property name="default_base_rot" value="0 0 0"/>
     <!--xacro:macro name="jaco_robot" params="parent prefix"-->
     <xacro:macro name="j2s7s300" params="base_parent prefix:=j2s7s300 trans:=${default_base_trans} rot:=${default_base_rot}">
