Commit message: Bring back the old xacro, but with the new joint limits

File: kinova_description/urdf/j2s7s300.xacro (robot description, xacro)
@@ -15,15 +15,15 @@
     xmlns:xacro="http://ros.org/wiki/xacro">
     <xacro:include filename="$(find kinova_description)/urdf/kinova_common.xacro" />
-    <xacro:include filename="$(find kinova_description)/urdf/kinova_finger_set.xacro" />
+    <xacro:include filename="$(find robotiq_85_description)/urdf/robotiq_85_gripper.urdf.xacro" />
     <!-- Import all Gazebo-customization elements -->
     <xacro:include filename="$(find kinova_description)/urdf/kinova.gazebo" />
-    <property name="link_base_mesh" value="base" />
-    <property name="link_1_mesh" value="shoulder" />
-    <property name="link_2_mesh" value="arm_half_1" />
-    <property name="link_3_mesh" value="arm_half_2" />
-    <property name="link_4_mesh" value="forearm" />
-    <property name="link_5_mesh" value="wrist_spherical_1" />
-    <property name="link_6_mesh" value="wrist_spherical_2" />
-    <property name="link_7_mesh" value="hand_3finger" />
+    <xacro:property name="link_base_mesh" value="base" />
+    <xacro:property name="link_1_mesh" value="shoulder" />
+    <xacro:property name="link_2_mesh" value="arm_half_1" />
+    <xacro:property name="link_3_mesh" value="arm_half_2" />
+    <xacro:property name="link_4_mesh" value="forearm" />
+    <xacro:property name="link_5_mesh" value="wrist_spherical_1" />
+    <xacro:property name="link_6_mesh" value="wrist_spherical_2" />
+    <xacro:property name="link_7_mesh" value="hand_3finger" />
     <!--Used for conditional arguments for setting inertial parameters
         base 0, shoulder 1, arm 2, forearm 3, wrist 4, arm_mico 5,
@@ -32,75 +32,76 @@
         hand 3 finger 55, hand_2finger 56, finger_proximal 57, finger_distal 58
     -->
-    <property name="link_base_mesh_no" value="0" />
-    <property name="link_1_mesh_no" value="1" />
-    <property name="link_2_mesh_no" value="6" />
-    <property name="link_3_mesh_no" value="7" />
-    <property name="link_4_mesh_no" value="3" />
-    <property name="link_5_mesh_no" value="8" />
-    <property name="link_6_mesh_no" value="9" />
-    <property name="link_7_mesh_no" value="55" />
-    <property name="joint_base" value="joint_base" />
-    <property name="joint_base_type" value="fixed" />
-    <property name="joint_base_axis_xyz" value="0 0 0" />
-    <property name="joint_base_origin_xyz" value="0 0 0" />
-    <property name="joint_base_origin_rpy" value="0 0 0" />
-    <property name="joint_1" value="joint_1" />
-    <property name="joint_1_type" value="continuous" />
-    <property name="joint_1_axis_xyz" value="0 0 1" />
-    <property name="joint_1_origin_xyz" value="0 0 0.15675" />
-    <property name="joint_1_origin_rpy" value="0 ${J_PI} 0" />
-    <property name="joint_1_lower_limit" value="${-2*J_PI}" />
-    <property name="joint_1_upper_limit" value="${2*J_PI}" />
-    <property name="joint_2" value="joint_2" />
-    <property name="joint_2_type" value="revolute" />
-    <property name="joint_2_axis_xyz" value="0 0 1" />
-    <property name="joint_2_origin_xyz" value="0 0.0016 -0.11875" />
-    <property name="joint_2_origin_rpy" value="-${J_PI/2} 0 ${J_PI}" />
-    <property name="joint_2_lower_limit" value="${47/180*J_PI}" />
-    <property name="joint_2_upper_limit" value="${313/180*J_PI}" />
-    <property name="joint_3" value="joint_3" />
-    <property name="joint_3_type" value="continuous" />
-    <property name="joint_3_axis_xyz" value="0 0 1" />
-    <property name="joint_3_origin_xyz" value="0 -0.205 0" />
-    <property name="joint_3_origin_rpy" value="-${J_PI/2} 0 0" />
-    <property name="joint_3_lower_limit" value="${-2*J_PI}" />
-    <property name="joint_3_upper_limit" value="${2*J_PI}" />
-    <property name="joint_4" value="joint_4" />
-    <property name="joint_4_type" value="revolute" />
-    <property name="joint_4_axis_xyz" value="0 0 1" />
-    <property name="joint_4_origin_xyz" value="0 0 -0.205" />
-    <property name="joint_4_origin_rpy" value="${J_PI/2} 0 ${J_PI}"/>
-    <property name="joint_4_lower_limit" value="${30/180*J_PI}" />
-    <property name="joint_4_upper_limit" value="${330/180*J_PI}" />
-    <property name="joint_5" value="joint_5" />
-    <property name="joint_5_type" value="continuous" />
-    <property name="joint_5_axis_xyz" value="0 0 1" />
-    <property name="joint_5_origin_xyz" value="0 0.2073 -0.0114" />
-    <property name="joint_5_origin_rpy" value="${-J_PI/2} 0 ${J_PI}" />
-    <property name="joint_5_lower_limit" value="${-2*J_PI}" />
-    <property name="joint_5_upper_limit" value="${2*J_PI}" />
-    <property name="joint_6" value="joint_6" />
-    <property name="joint_6_type" value="revolute" />
-    <property name="joint_6_axis_xyz" value="0 0 1" />
-    <property name="joint_6_origin_xyz" value="0 0 -0.10375" />
-    <property name="joint_6_origin_rpy" value="${J_PI/2} 0 ${J_PI}" />
-    <property name="joint_6_lower_limit" value="${65/180*J_PI}" />
-    <property name="joint_6_upper_limit" value="${295/180*J_PI}" />
-    <property name="joint_7" value="joint_7" />
-    <property name="joint_7_type" value="continuous" />
-    <property name="joint_7_axis_xyz" value="0 0 1" />
-    <property name="joint_7_origin_xyz" value="0 0.10375 0" />
-    <property name="joint_7_origin_rpy" value="${-J_PI/2} 0 ${J_PI}" />
-    <property name="joint_7_lower_limit" value="${-2*J_PI}" />
-    <property name="joint_7_upper_limit" value="${2*J_PI}" />
-    <property name="joint_end_effector" value="end_effector_offset" />
-    <property name="joint_end_effector_type" value="fixed" />
-    <property name="joint_end_effector_axis_xyz" value="0 0 0" />
-    <property name="joint_end_effector_origin_xyz" value="0 0 -0.1600" />
-    <property name="joint_end_effector_origin_rpy" value="${J_PI} 0 0" />
-    <xacro:macro name="j2s7s300" params="base_parent prefix:=j2s7s300">
+    <xacro:property name="link_base_mesh_no" value="0" />
+    <xacro:property name="link_1_mesh_no" value="1" />
+    <xacro:property name="link_2_mesh_no" value="6" />
+    <xacro:property name="link_3_mesh_no" value="7" />
+    <xacro:property name="link_4_mesh_no" value="3" />
+    <xacro:property name="link_5_mesh_no" value="8" />
+    <xacro:property name="link_6_mesh_no" value="9" />
+    <xacro:property name="link_7_mesh_no" value="55" />
+    <xacro:property name="joint_base" value="joint_base" />
+    <xacro:property name="joint_base_type" value="fixed" />
+    <xacro:property name="joint_base_axis_xyz" value="0 0 0" />
+    <xacro:property name="joint_1" value="joint_1" />
+    <xacro:property name="joint_1_type" value="continuous" />
+    <xacro:property name="joint_1_axis_xyz" value="0 0 1" />
+    <xacro:property name="joint_1_origin_xyz" value="0 0 0.15675" />
+    <xacro:property name="joint_1_origin_rpy" value="0 ${J_PI} 0" />
+    <xacro:property name="joint_1_lower_limit" value="${-2*J_PI}" />
+    <xacro:property name="joint_1_upper_limit" value="${2*J_PI}" />
+    <xacro:property name="joint_2" value="joint_2" />
+    <xacro:property name="joint_2_type" value="revolute" />
+    <xacro:property name="joint_2_axis_xyz" value="0 0 1" />
+    <xacro:property name="joint_2_origin_xyz" value="0 0.0016 -0.11875" />
+    <xacro:property name="joint_2_origin_rpy" value="-${J_PI/2} 0 ${J_PI}" />
+    <xacro:property name="joint_2_lower_limit" value="${47/180*J_PI}" />
+    <xacro:property name="joint_2_upper_limit" value="${313/180*J_PI}" />
+    <xacro:property name="joint_3" value="joint_3" />
+    <xacro:property name="joint_3_type" value="continuous" />
+    <xacro:property name="joint_3_axis_xyz" value="0 0 1" />
+    <xacro:property name="joint_3_origin_xyz" value="0 -0.205 0" />
+    <xacro:property name="joint_3_origin_rpy" value="-${J_PI/2} 0 0" />
+    <xacro:property name="joint_3_lower_limit" value="${-2*J_PI}" />
+    <xacro:property name="joint_3_upper_limit" value="${2*J_PI}" />
+    <xacro:property name="joint_4" value="joint_4" />
+    <xacro:property name="joint_4_type" value="revolute" />
+    <xacro:property name="joint_4_axis_xyz" value="0 0 1" />
+    <xacro:property name="joint_4_origin_xyz" value="0 0 -0.205" />
+    <xacro:property name="joint_4_origin_rpy" value="${J_PI/2} 0 ${J_PI}"/>
+    <xacro:property name="joint_4_lower_limit" value="${30/180*J_PI}" />
+    <xacro:property name="joint_4_upper_limit" value="${330/180*J_PI}" />
+    <xacro:property name="joint_5" value="joint_5" />
+    <xacro:property name="joint_5_type" value="continuous" />
+    <xacro:property name="joint_5_axis_xyz" value="0 0 1" />
+    <xacro:property name="joint_5_origin_xyz" value="0 0.2073 -0.0114" />
+    <xacro:property name="joint_5_origin_rpy" value="${-J_PI/2} 0 ${J_PI}" />
+    <xacro:property name="joint_5_lower_limit" value="${-2*J_PI}" />
+    <xacro:property name="joint_5_upper_limit" value="${2*J_PI}" />
+    <xacro:property name="joint_6" value="joint_6" />
+    <xacro:property name="joint_6_type" value="revolute" />
+    <xacro:property name="joint_6_axis_xyz" value="0 0 1" />
+    <xacro:property name="joint_6_origin_xyz" value="0 0 -0.10375" />
+    <xacro:property name="joint_6_origin_rpy" value="${J_PI/2} 0 ${J_PI}" />
+    <xacro:property name="joint_6_lower_limit" value="${65/180*J_PI}" />
+    <xacro:property name="joint_6_upper_limit" value="${295/180*J_PI}" />
+    <xacro:property name="joint_7" value="joint_7" />
+    <xacro:property name="joint_7_type" value="continuous" />
+    <xacro:property name="joint_7_axis_xyz" value="0 0 1" />
+    <xacro:property name="joint_7_origin_xyz" value="0 0.10375 0" />
+    <xacro:property name="joint_7_origin_rpy" value="${-J_PI/2} 0 ${J_PI}" />
+    <xacro:property name="joint_7_lower_limit" value="${-2*J_PI}" />
+    <xacro:property name="joint_7_upper_limit" value="${2*J_PI}" />
+    <xacro:property name="joint_end_effector" value="end_effector_offset" />
+    <xacro:property name="joint_end_effector_type" value="fixed" />
+    <xacro:property name="joint_end_effector_axis_xyz" value="0 0 0" />
+    <xacro:property name="joint_end_effector_origin_xyz" value="0 0 -0.1600" />
+    <xacro:property name="joint_end_effector_origin_rpy" value="${J_PI} 0 0" />
+    <!--xacro:macro name="jaco_robot" params="parent prefix"-->
+    <xacro:property name="default_base_trans" value="0 0 0" />
+    <xacro:property name="default_base_rot" value="0 0 0" />
+    <xacro:macro name="j2s7s300" params="base_parent prefix:=j2s7s300 trans:=${default_base_trans} rot:=${default_base_rot}">
         <xacro:gazebo_config robot_namespace="${prefix}"/>
         <xacro:kinova_armlink link_name="${prefix}_link_base" link_mesh="${link_base_mesh}" mesh_no="${link_base_mesh_no}"/>
-        <xacro:kinova_armjoint joint_name="${prefix}_joint_base" type="${joint_base_type}" parent="${base_parent}" child="${prefix}_link_base" joint_axis_xyz="${joint_base_axis_xyz}" joint_origin_xyz="${joint_base_origin_xyz}" joint_origin_rpy="${joint_base_origin_rpy}" joint_lower_limit="0" joint_upper_limit="0" fixed="true"/>
+        <xacro:kinova_armjoint joint_name="${prefix}_joint_base" type="${joint_base_type}" parent="${base_parent}" child="${prefix}_link_base" joint_axis_xyz="${joint_base_axis_xyz}" joint_origin_xyz="${trans}" joint_origin_rpy="${rot}" joint_lower_limit="0" joint_upper_limit="0" fixed="true"/>
         <xacro:kinova_armlink link_name="${prefix}_link_1" link_mesh="${link_1_mesh}" use_ring_mesh="true" mesh_no="${link_1_mesh_no}"/>
         <xacro:kinova_armjoint joint_name="${prefix}_joint_1" type="${joint_1_type}" parent="${prefix}_link_base" child="${prefix}_link_1" joint_axis_xyz="${joint_1_axis_xyz}" joint_origin_xyz="${joint_1_origin_xyz}" joint_origin_rpy="${joint_1_origin_rpy}" joint_lower_limit="${joint_1_lower_limit}" joint_upper_limit="${joint_1_upper_limit}"/>
@@ -115,4 +116,5 @@
         <xacro:kinova_armlink link_name="${prefix}_link_6" link_mesh="${link_6_mesh}" use_ring_mesh="true" ring_mesh="ring_small" mesh_no="${link_6_mesh_no}"/>
         <xacro:kinova_armjoint joint_name="${prefix}_joint_6" type="${joint_6_type}" parent="${prefix}_link_5" child="${prefix}_link_6" joint_axis_xyz="${joint_6_axis_xyz}" joint_origin_xyz="${joint_6_origin_xyz}" joint_origin_rpy="${joint_6_origin_rpy}" joint_lower_limit="${joint_6_lower_limit}" joint_upper_limit="${joint_6_upper_limit}"/>
+        <!--
         <xacro:kinova_armlink link_name="${prefix}_link_7" link_mesh="${link_7_mesh}" use_ring_mesh="true" ring_mesh="ring_small" mesh_no="${link_7_mesh_no}"/>
         <xacro:kinova_armjoint joint_name="${prefix}_joint_7" type="${joint_7_type}" parent="${prefix}_link_6" child="${prefix}_link_7" joint_axis_xyz="${joint_7_axis_xyz}" joint_origin_xyz="${joint_7_origin_xyz}" joint_origin_rpy="${joint_7_origin_rpy}" joint_lower_limit="${joint_7_lower_limit}" joint_upper_limit="${joint_7_upper_limit}"/>
@@ -120,4 +122,50 @@
         <xacro:kinova_virtual_joint joint_name="${prefix}_joint_end_effector" type="${joint_end_effector_type}" parent="${prefix}_link_7" child="${prefix}_end_effector" joint_axis_xyz="${joint_end_effector_axis_xyz}" joint_origin_xyz="${joint_end_effector_origin_xyz}" joint_origin_rpy="${joint_end_effector_origin_rpy}" joint_lower_limit="0" joint_upper_limit="0"/>
         <xacro:kinova_3fingers link_hand="${prefix}_link_7" prefix="${prefix}_"/>
+        -->
+        <!-- RAIL end-effector additions/modifications -->
+        <joint name="${prefix}_joint_7" type="continuous">
+          <parent link="${prefix}_link_6" />
+          <child link = "${prefix}_link_7" />
+          <origin xyz="0 0.06075 0" rpy="${J_PI/2} 0 0" />
+          <axis xyz="0 0 1" />
+          <limit effort="600.8" velocity="0.785"/>
+          <dynamics damping="0.0" friction="0.0"/>
+        </joint>
+        <link name="${prefix}_link_7">
+          <visual>
+            <geometry>
+              <mesh filename="package://kinova_description/meshes/wrist_3.dae"/>
+            </geometry>
+          </visual>
+          <collision>
+            <geometry>
+              <mesh filename="package://kinova_description/meshes/wrist_3.stl"/>
+            </geometry>
+          </collision>
+        </link>
+        <joint name="${prefix}_ee_fixed_joint" type="fixed">
+          <parent link="${prefix}_link_7" />
+          <child link = "${prefix}_ee_base" />
+          <origin xyz="0 0 -0.09380704" rpy="0 ${J_PI/2} 0" />
+        </joint>
+        <link name="${prefix}_ee_base"/>
+        <joint name="${prefix}_ee_gripper" type="fixed">
+          <parent link="${prefix}_ee_base" />
+          <child link ="${prefix}_ee_link" />
+          <origin xyz="0.13 0 0" />
+        </joint>
+        <link name="${prefix}_ee_link"/>
+        <transmission name="${prefix}_joint_7_trans">
+          <type>transmission_interface/SimpleTransmission</type>
+          <joint name="${prefix}_joint_7">
+            <hardwareInterface>PositionJointInterface</hardwareInterface>
+          </joint>
+          <actuator name="${prefix}_joint_7_actuator">
+            <mechanicalReduction>160</mechanicalReduction>
+          </actuator>
+        </transmission>
+        <xacro:robotiq_85_gripper prefix="" parent="${prefix}_ee_base">
+          <origin xyz="0 0 0" rpy="${J_PI/2} 0 0" />
+        </xacro:robotiq_85_gripper>
     </xacro:macro>
 </root>
